File: Schematic_withShiftResister.brd (EAGLE design)
At the start: 100 x 80 mm, 39 parts, among them U1 328P, U3 3.3V/150mA, U5 SN74HC595N, U6 SN74HC595N

Commit message: Add files via upload
Parts:
- moved Y 2.18 mm to (68.6, 72.5)
- moved X 2.17 mm to (68.7, 75.1)
- moved Z 2.14 mm to (68.6, 69.9)
- moved 0G 2.08 mm to (68.6, 64.7)
- moved SL 2.04 mm to (68.6, 67.2)
Routing:
- net N$18: track 93.3 -> 91.0 mm
- net N$17: track 95.5 -> 93.4 mm
- net N$19: track 89.7 -> 87.6 mm
- net N$42: track 114.4 -> 116.4 mm
- net N$41: track 90.1 -> 92.1 mm
Changed lines of the file:
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@@
 </autorouter>
 <elements>
-<element name="0G" library="adafruit" library_urn="urn:adsk.eagle:library:420" package="1X01" value="" x="70.67905" y="64.7026875" smashed="yes">
-<attribute name="NAME" x="67.029640625" y="64.227328125" size="1.27" layer="25" ratio="10"/>
-<attribute name="VALUE" x="69.40905" y="61.5276875" size="1.27" layer="27"/>
+<element name="0G" library="adafruit" library_urn="urn:adsk.eagle:library:420" package="1X01" value="" x="68.595296875" y="64.7026875" smashed="yes">
+<attribute name="NAME" x="64.9458875" y="64.227328125" size="1.27" layer="25" ratio="10"/>
+<attribute name="VALUE" x="67.325296875" y="61.5276875" size="1.27" layer="27"/>
 </element>
 <element name="3.3V" library="adafruit" library_urn="urn:adsk.eagle:library:420" package="1X01" value="" x="93.751775" y="72.273159375" smashed="yes">
@@
 <attribute name="SF_SKU" value="COM-00097" x="21.736240625" y="20.583015625" size="1.778" layer="27" rot="R270" display="off"/>
 </element>
-<element name="SL" library="adafruit" library_urn="urn:adsk.eagle:library:420" package="1X01" value="" x="70.685915625" y="67.243834375" smashed="yes">
-<attribute name="NAME" x="67.430396875" y="66.768471875" size="1.27" layer="25" ratio="10"/>
-<attribute name="VALUE" x="69.415915625" y="64.068834375" size="1.27" layer="27"/>
+<element name="SL" library="adafruit" library_urn="urn:adsk.eagle:library:420" package="1X01" value="" x="68.646484375" y="67.243834375" smashed="yes">
+<attribute name="NAME" x="65.390965625" y="66.768471875" size="1.27" layer="25" ratio="10"/>
+<attribute name="VALUE" x="67.376484375" y="64.068834375" size="1.27" layer="27"/>
 </element>
 <element name="ST" library="adafruit" library_urn="urn:adsk.eagle:library:420" package="1X01" value="" x="93.8084875" y="64.43566875" smashed="yes">
@@
 <attribute name="PROD_ID" value="IC-13123" x="82.8287" y="45.834428125" size="1.778" layer="27" rot="R180" display="off"/>
 </element>
-<element name="X" library="adafruit" library_urn="urn:adsk.eagle:library:420" package="1X01" value="" x="70.835075" y="74.970765625" smashed="yes">
-<attribute name="NAME" x="68.218875" y="74.41685625" size="1.27" layer="25" ratio="10"/>
-<attribute name="VALUE" x="69.565075" y="71.795765625" size="1.27" layer="27"/>
-</element>
-<element name="Y" library="adafruit" library_urn="urn:adsk.eagle:library:420" package="1X01" value="" x="70.794434375" y="72.36656875" smashed="yes">
-<attribute name="NAME" x="68.440171875" y="71.824659375" size="1.27" layer="25" ratio="10"/>
-<attribute name="VALUE" x="69.524434375" y="69.19156875" size="1.27" layer="27"/>
-</element>
-<element name="Z" library="adafruit" library_urn="urn:adsk.eagle:library:420" package="1X01" value="" x="70.75373125" y="69.69665" smashed="yes">
-<attribute name="NAME" x="68.104384375" y="69.130359375" size="1.27" layer="25" ratio="10"/>
-<attribute name="VALUE" x="69.48373125" y="66.52165" size="1.27" layer="27"/>
+<element name="X" library="adafruit" library_urn="urn:adsk.eagle:library:420" package="1X01" value="" x="68.662675" y="75.0594125" smashed="yes">
+<attribute name="NAME" x="66.046475" y="74.505503125" size="1.27" layer="25" ratio="10"/>
+<attribute name="VALUE" x="67.392675" y="71.8844125" size="1.27" layer="27"/>
+</element>
+<element name="Y" library="adafruit" library_urn="urn:adsk.eagle:library:420" package="1X01" value="" x="68.6220375" y="72.499603125" smashed="yes">
+<attribute name="NAME" x="66.267775" y="71.95769375" size="1.27" layer="25" ratio="10"/>
+<attribute name="VALUE" x="67.3520375" y="69.324603125" size="1.27" layer="27"/>
+</element>
+<element name="Z" library="adafruit" library_urn="urn:adsk.eagle:library:420" package="1X01" value="" x="68.625653125" y="69.918328125" smashed="yes">
+<attribute name="NAME" x="65.97630625" y="69.3520375" size="1.27" layer="25" ratio="10"/>
+<attribute name="VALUE" x="67.355653125" y="66.743328125" size="1.27" layer="27"/>
 </element>
 <element name="C4" library="adafruit" library_urn="urn:adsk.eagle:library:420" package="C0805" value="0.1uF" x="52.597878125" y="22.23280625" smashed="yes" rot="R90">
@@
 <via x="11.0851875" y="37.134853125" extent="1-16" drill="0.35"/>
 <via x="26.78893125" y="18.667528125" extent="1-16" drill="0.35"/>
+<via x="79.804759375" y="70.350621875" extent="1-16" drill="0.35"/>
+<via x="76.147475" y="77.459321875" extent="1-16" drill="0.35"/>
+<via x="63.822253125" y="76.350740625" extent="1-16" drill="0.35"/>
+<via x="67.236078125" y="49.390609375" extent="1-16" drill="0.35"/>
 </signal>
 <signal name="MISO">
@@
 <wire x1="60.350528125" y1="51.4454125" x2="60.350528125" y2="73.94854375" width="0.3556" layer="1"/>
 <wire x1="60.350528125" y1="73.94854375" x2="61.37275" y2="74.970765625" width="0.3556" layer="1"/>
-<wire x1="61.37275" y1="74.970765625" x2="70.835075" y2="74.970765625" width="0.3556" layer="1"/>
+<wire x1="61.37275" y1="74.970765625" x2="68.662675" y2="75.0594125" width="0.3556" layer="1"/>
 </signal>
 <signal name="N$18">
 <contactref element="Y" pad="1"/>
 <contactref element="U1" pad="24"/>
-<wire x1="70.794434375" y1="72.36656875" x2="70.56805625" y2="72.592946875" width="0.3556" layer="1"/>
-<wire x1="70.56805625" y1="72.592946875" x2="63.46628125" y2="72.592946875" width="0.3556" layer="1"/>
-<wire x1="63.46628125" y1="72.592946875" x2="61.84068125" y2="70.967346875" width="0.3556" layer="1"/>
+<wire x1="61.84068125" y1="70.967346875" x2="63.46628125" y2="72.592946875" width="0.3556" layer="1"/>
 <wire x1="61.84068125" y1="70.967346875" x2="61.84068125" y2="49.27644375" width="0.3556" layer="1"/>
 <wire x1="61.84068125" y1="49.27644375" x2="61.976128125" y2="49.411890625" width="0.3556" layer="1"/>
@@
 <wire x1="72.00944375" y1="38.59974375" x2="73.218040625" y2="38.59974375" width="0.3556" layer="16"/>
 <wire x1="73.218040625" y1="38.59974375" x2="77.202221875" y2="34.6155625" width="0.3556" layer="16"/>
-<wire x1="77.202221875" y1="34.6155625" x2="77.202221875" y2="25.73610625" width="0.3556" layer="16"/>
-<wire x1="77.202221875" y1="25.73610625" x2="77.202221875" y2="25.6025" width="0.3556" layer="16"/>
-<wire x1="77.202221875" y1="25.73610625" x2="77.202221875" y2="20.954175" width="0.3556" layer="16"/>
+<wire x1="77.202221875" y1="34.6155625" x2="77.202221875" y2="20.954175" width="0.3556" layer="16"/>
 <wire x1="63.21551875" y1="20.137184375" x2="63.168465625" y2="20.09013125" width="0.3556" layer="16"/>
 <via x="63.168465625" y="20.09013125" extent="1-16" drill="0.3556"/>
@@
 <wire x1="77.202221875" y1="20.954175" x2="76.38523125" y2="20.137184375" width="0.3556" layer="16"/>
 <wire x1="76.38523125" y1="20.137184375" x2="63.21551875" y2="20.137184375" width="0.3556" layer="16"/>
+<wire x1="63.46628125" y1="72.592946875" x2="68.52869375" y2="72.592946875" width="0.254" layer="1"/>
+<wire x1="68.52869375" y1="72.592946875" x2="68.6220375" y2="72.499603125" width="0.1524" layer="1"/>
 </signal>
 <signal name="N$19">
 <contactref element="Z" pad="1"/>
 <contactref element="U1" pad="25"/>
-<wire x1="70.75373125" y1="69.69665" x2="63.843475" y2="69.69665" width="0.3556" layer="1"/>
+<wire x1="68.625653125" y1="69.918328125" x2="63.843475" y2="69.69665" width="0.3556" layer="1"/>
 <wire x1="63.843475" y1="69.69665" x2="63.262575" y2="69.11575" width="0.3556" layer="1"/>
 <wire x1="63.262575" y1="69.11575" x2="63.262575" y2="50.6723" width="0.3556" layer="1"/>
@@
 <contactref element="SL" pad="1"/>
 <contactref element="U1" pad="26"/>
-<wire x1="70.685915625" y1="67.243834375" x2="83.84508125" y2="67.243834375" width="0.3556" layer="16"/>
+<wire x1="68.646484375" y1="67.243834375" x2="83.84508125" y2="67.243834375" width="0.3556" layer="16"/>
 <via x="94.001715625" y="43.929553125" extent="1-16" drill="0.3556"/>
 <wire x1="94.001715625" y1="43.929553125" x2="94.001715625" y2="40.372284375" width="0.3556" layer="1"/>
@@
 <via x="78.029053125" y="64.592390625" extent="1-16" drill="0.3556"/>
 <wire x1="78.029053125" y1="64.592390625" x2="70.789346875" y2="64.592390625" width="0.3556" layer="16"/>
-<wire x1="70.789346875" y1="64.592390625" x2="70.67905" y2="64.7026875" width="0.3556" layer="16"/>
+<wire x1="70.789346875" y1="64.592390625" x2="68.595296875" y2="64.7026875" width="0.3556" layer="16"/>
 <wire x1="98.066734375" y1="28.796425" x2="98.066734375" y2="74.637071875" width="0.3556" layer="1"/>
 </signal>
