File: Schematic_withShiftResister.brd (EAGLE design)
At the start: 100 x 80 mm, 39 parts, among them U1 328P, U3 3.3V/150mA, U5 SN74HC595N, U6 SN74HC595N

Commit message: Add files via upload
Connections:
- new net S$1: R4.2
- net N$4: no longer R4.2
Routing:
- net N$4: track 41.8 -> 30.6 mm, vias 2 -> 0
- net S$1: track 0.00 -> 10.6 mm, vias 0 -> 1
Changed lines of the file:
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@@
 <wire x1="58.301825" y1="45.268175" x2="58.42" y2="45.15" width="0.3556" layer="16"/>
 </signal>
-<signal name="N$4">
-<contactref element="LED-MATRIX" pad="12"/>
-<contactref element="R4" pad="2"/>
-<via x="74.894121875" y="62.402909375" extent="1-16" drill="0.3556"/>
-<wire x1="78.342934375" y1="62.402909375" x2="74.894121875" y2="62.402909375" width="0.3556" layer="16"/>
+<signal name="S$1">
 <wire x1="78.342934375" y1="62.402909375" x2="78.3821125" y2="62.36373125" width="0.3556" layer="16"/>
 <wire x1="78.3821125" y1="62.36373125" x2="78.421290625" y2="62.402909375" width="0.3556" layer="16"/>
@@
 <via x="78.4605375" y="62.402909375" extent="1-16" drill="0.3556"/>
 <wire x1="78.4605375" y1="62.402909375" x2="84.111528125" y2="56.75191875" width="0.3556" layer="1"/>
+<contactref element="R4" pad="2"/>
 <wire x1="84.111528125" y1="56.75191875" x2="84.111528125" y2="54.271534375" width="0.3556" layer="1"/>
-<wire x1="74.894121875" y1="62.402909375" x2="67.28435" y2="62.402909375" width="0.3556" layer="16"/>
+</signal>
+<signal name="N$4">
+<contactref element="LED-MATRIX" pad="12"/>
 <wire x1="62.652340625" y1="67.03491875" x2="51.409728125" y2="67.03491875" width="0.3556" layer="16"/>
 <wire x1="51.409728125" y1="67.03491875" x2="50.8" y2="67.644646875" width="0.3556" layer="16"/>
 <wire x1="50.8" y1="67.644646875" x2="50.8" y2="69.15" width="0.3556" layer="16"/>
-<wire x1="67.28435" y1="62.402909375" x2="62.652340625" y2="67.03491875" width="0.3556" layer="16"/>
+<wire x1="62.652340625" y1="67.03491875" x2="67.28435" y2="62.402909375" width="0.3556" layer="16"/>
+<wire x1="67.28435" y1="62.402909375" x2="77.72393125" y2="62.402909375" width="0.254" layer="16"/>
 </signal>
 <signal name="N$5">
@@
 </signal>
 </signals>
+<errors>
+</errors>
 </board>
 </drawing>
