File: Schematic_withShiftResister.sch (EAGLE design)
At the start: 31 parts, among them U1 328P, U2 SN74HC595D, U3 3.3V/150mA, U4 SN74HC595D

Commit message: Add files via upload
Parts:
- removed AA/18650: (no value), SparkFun-Batteries:BATTERY-9V
- removed C5: 22pF, adafruit:C-US025-024X044
- added BT1: (no value), SparkFun-Retired:BATTERYAA-PANEL
- added C10: 0.1uF, SparkFun-Capacitors:0.1UF-0402-16V-10%
- C1: value 2.2uF -> 0.1uF; device adafruit:C-US025-024X044 -> SparkFun-Capacitors:0.1UF-0402-16V-10%; MPN 12105C225K4Z2A -> (none); OC_NEWARK 85Y0347 -> (none)
- C2: value 470pF -> 2.2uF; device adafruit:C-US025-024X044 -> SparkFun-Capacitors:2.2UF-0603-10V-20%; OC_NEWARK unknown -> (none)
- C3, C6, C8: device adafruit:C-US025-024X044 -> SparkFun-Capacitors:0.1UF-0402-16V-10%; OC_NEWARK unknown -> (none)
- C4: device adafruit:C-US025-024X044 -> SparkFun-Capacitors:22PF-0603-50V-5%; OC_NEWARK unknown -> (none)
- C7: value 0.1uF -> 22pF; device adafruit:C-US025-024X044 -> SparkFun-Capacitors:22PF-0603-50V-5%; OC_NEWARK unknown -> (none)
- C9: value 0.1uF -> 470pF; device adafruit:C-US025-024X044 -> SparkFun-Capacitors:470PF-0603-50V-5%; OC_NEWARK unknown -> (none)
- R1, R2, R3, R4, R5, R6, R8: value 120 -> 150; device SparkFun-Resistors:0.1OHM-1210-1/2W-1% -> SparkFun-Resistors:150OHM-0603-1/10W-1%; OC_NEWARK unknown -> (none)
- R7: value 120 -> 150; device SparkFun-Resistors:0.1OHM-1210-1/2W-1% -> SparkFun-Resistors:150OHM-0603-1/10W-1%; OC_NEWARK unknown -> (none); SPICEPREFIX R -> (none)
- R9: value 120 -> 150; device SparkFun-Resistors:200OHM-0603-1/10W-1% -> SparkFun-Resistors:150OHM-0603-1/10W-1%; OC_NEWARK unknown -> (none)
Connections:
- net +3.3V: now also C10.1, C2.1; no longer C7.1, C9.1
- net GND: now also BT1.-, C10.2, C7.1; no longer AA/18650.-, C5.1, C7.2
- net N$30: now also C4.2; no longer C5.2
- net N$31: now also C7.2; no longer C4.2
- net N$32: now also C9.1; no longer C2.1
- net N$36: now also BT1.+; no longer AA/18650.+
Other:
- moved on the sheet: C1, C2, C4, C6, C7, C8, C9, R1

Commit message: Add files via upload
Parts:
- removed C4, C7: 22pF, SparkFun-Capacitors:22PF-0603-50V-5%
- removed C6: 0.1uF, SparkFun-Capacitors:0.1UF-0402-16V-10%
- removed LED1: (no value), adafruit:LED
- removed Q1: (no value), adafruit:CRYSTALHC49S
- removed R9: 150, SparkFun-Resistors:150OHM-0603-1/10W-1%
- removed U$2: MMA7361, SparkFun:MMA7361
- removed U2, U4: SN74HC595D, SparkFun-IC-Logic:74HC595D
- added 0G, 3.3V, 5V, GND, GS, SL, ST, X, Y, Z: (no value), adafruit:PINHD-1X1
- added BT2, BT3: (no value), SparkFun-Batteries:BATTERY-AAA_KIT
- added C5: 0.1uF, SparkFun-Capacitors:0.1UF-0402-16V-10%
- added R10, R11: 10k, SparkFun-Resistors:10KOHM-0603-1/10W-1%
- added U5, U6: SN74HC595N, SparkFun-IC-Logic:74HC595N
- BT1: device SparkFun-Retired:BATTERYAA-PANEL -> SparkFun-Batteries:BATTERY-AAA_KIT
Connections:
- removed net +3.3V: C1.1, C10.1, C2.1, C6.1, C8.1, ISP.VCC, L2.1, U$2.VDD, U1.PB0(ICP), U1.PB1(OC1A), U1.PD4(XCK/T0), U1.PD5(T1), U1.VCC, U2.SCL, U2.VCC, U3.OUT, U4.SCL, U4.VCC
- removed net N$37: R9.2, U1.PD7(AIN1)
- removed net N$39: LED1.A, R9.1
- removed net N$44: U$2.GSELECT, U1.PC5(ADC5/SCL)
- new net 3.3V: 3.3V.1, C1.1, C10.1, C2.1, C8.1, ISP.VCC, L2.1, R10.2, R11.2, U1.VCC, U3.OUT, U5.SCL, U5.VCC, U6.SCL, U6.VCC
- new net N$46: ST.1, U1.PD4(XCK/T0)
- net GND: now also 5V.1, BT3.-, C5.1, GND.1, U5.G, U5.GND, U6.G, U6.GND; no longer BT1.-, C4.1, C6.2, C7.1, LED1.C, U$2.VSS, U2.G, U2.GND, U4.G, U4.GND
- net N$10: now also U5.QC; no longer U4.QC
- net N$11: now also U5.QD; no longer U4.QD
- net N$12: now also U5.QE; no longer U4.QE
- net N$13: now also U5.QF; no longer U4.QF
- net N$14: now also U5.QG; no longer U4.QG
- net N$15: now also U5.QH; no longer U4.QH
- net N$16: now also U6.QA; no longer U2.QA
- net N$17: now also X.1; no longer U$2.XOUT
- net N$18: now also Y.1; no longer U$2.YOUT
- net N$19: now also Z.1; no longer U$2.ZOUT
- net N$20: now also U6.QB; no longer U2.QB
- net N$21: now also U6.QC; no longer U2.QC
- net N$22: now also U6.QD; no longer U2.QD
- net N$23: now also U6.QE; no longer U2.QE
- net N$24: now also U6.QF; no longer U2.QF
- net N$25: now also U6.QG; no longer U2.QG
- net N$26: now also U6.QH; no longer U2.QH
- net N$27: now also U5.QB; no longer U4.QB
- net N$28: now also U5.SCK, U6.SCK; no longer U2.SCK, U4.SCK
- net N$30: now also BT2.-, BT3.+; no longer C4.2, Q1.2, U1.PB7(XTAL2/TOSC2)
- net N$31: now also BT1.-, BT2.+; no longer C7.2, Q1.1, U1.PB6(XTAL1/TOSC1)
- net N$33: now also U5.SER; no longer U4.SER
- net N$34: now also U5.QH*, U6.SER; no longer U2.SER, U4.QH*
- net N$35: now also U5.RCK, U6.RCK; no longer U2.RCK, U4.RCK
- net N$38: now also C5.2, U1.AREF; no longer U1.PB5(SCK)
- net N$40: now also R11.1, U1.PD3(INT1); no longer U1.PD6(AIN0)
- net N$41: now also SL.1; no longer U$2.SLEEP
- net N$42: now also 0G.1; no longer U$2.0GD
- net N$45: now also GS.1, U1.PC5(ADC5/SCL); no longer U$2.ST, U1.PD3(INT1)
- net N$9: now also U5.QA; no longer U4.QA
- net RESET: now also R10.1
- net SCK: now also U1.PB5(SCK)
Other:
- note added: "1.5V AA Battery"
- note added: "Unused gpio pins - leave them float and make them output."
- note added: "Using Internal Crystal"
- note removed: "9V Battery"
- note removed: "MMA7361 Accelerometer"
- note removed: "Start LED"
- moved on the sheet: BT1, S1, U3

Commit message: Add files via upload
Parts:
- removed C5: 0.1uF, SparkFun-Capacitors:0.1UF-0402-16V-10%
- added C4: 0.1uF, adafruit:C-USC0805
- C1, C10, C3, C8: device SparkFun-Capacitors:0.1UF-0402-16V-10% -> adafruit:C-USC0805
- C2: device SparkFun-Capacitors:2.2UF-0603-10V-20% -> adafruit:C-USC0805
- C9: device SparkFun-Capacitors:470PF-0603-50V-5% -> adafruit:C-USC0805
Connections:
- new net N$37: C4.2, U1.AREF
- net 3.3V: no longer U5.SCL, U6.SCL
- net GND: now also C4.1; no longer C5.1
- net N$38: now also U1.PD5(T1), U5.SCL, U6.SCL; no longer C5.2, U1.AREF
Other:
- moved on the sheet: 0G, 3.3V, 5V, BT1, BT2, BT3, C1, C10, C2, C3, C8, C9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

Commit message: Add files via upload
Connections:
- net GND: no longer 5V.1
Changed lines of the file:
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@@
 </segment>
 <segment>
-<pinref part="5V" gate="G$1" pin="1"/>
-<wire x1="12.7" y1="66.04" x2="-7.62" y2="66.04" width="0.1524" layer="91"/>
-<wire x1="-7.62" y1="66.04" x2="-7.62" y2="55.88" width="0.1524" layer="91"/>
 <pinref part="GND10" gate="1" pin="GND"/>
 <pinref part="GND" gate="G$1" pin="1"/>
 <wire x1="-7.62" y1="55.88" x2="-7.62" y2="50.8" width="0.1524" layer="91"/>
 <wire x1="12.7" y1="55.88" x2="-7.62" y2="55.88" width="0.1524" layer="91"/>
-<junction x="-7.62" y="55.88"/>
 </segment>
 <segment>
